File: FSQCallTelemetry.brd (EAGLE design)
At the start: 53.3 x 49.5 mm, 22 parts, among them IC1 LM358, IC2 LM358, J1 1X2-3.5MM, J2 1X2-3.5MM, J3 1X2-3.5MM

Commit message: Add files via upload
Parts:
- added C3, C4: (no value), rcl:C050-025X075
- added JP1: (no value), jumper:JP1
- added R13: 100K, resistor:0207/10
- moved J1 0.89 mm to (48.1, 3.56)
- moved J3 0.89 mm to (34.2, 3.56)
Connections:
- new net N$26: JP1.2, R13.1
- new net N$6: C3.1, IC1.8, IC2.8, U$1.VIN
- new net N$7: C4.1, U$1.AREF
- net GND: now also C3.2, C4.2, R13.2
- net N$14: now also JP1.1
- net VCC: no longer IC1.8, IC2.8
Routing:
- net GND: track 171.2 -> 231.1 mm
- net N$6: track 0.00 -> 53.0 mm, vias 0 -> 2
- net N$26: track 0.00 -> 16.7 mm
- net VCC: track 99.0 -> 106.2 mm, vias 0 -> 3
- net N$7: track 0.00 -> 5.63 mm
- net N$14: track 56.6 -> 60.5 mm
- net N$17: track 43.1 -> 46.8 mm
- net N$19: track 25.9 -> 28.8 mm
- net N$2: track 38.2 -> 39.8 mm, vias 0 -> 1
- net N$10: track 53.8 -> 54.6 mm
- net N$21: track 61.7 -> 61.1 mm
Other:
- board text added: "FSQCall Telemetry Shield Rev A"
- board text removed: "FSQCall Telemetry Shield Rev --"

Commit message: FSQCall Rev B
Parts:
- moved JP1 0.56 mm to (21.3, 14.4)
Routing:
- net GND: track 231.1 -> 168.0 mm, vias 3 -> 0
- net N$1: track 82.2 -> 40.9 mm, vias 0 -> 1
- net N$14: track 60.5 -> 101.5 mm, vias 1 -> 0
- net N$10: track 54.6 -> 95.7 mm, vias 2 -> 0
- net N$15: track 34.6 -> 68.9 mm
- net N$18: track 53.0 -> 63.3 mm
- net N$17: track 46.8 -> 56.8 mm
- net N$2: track 39.8 -> 33.4 mm, vias 1 -> 0
- net VCC: track 106.2 -> 112.2 mm, vias 3 -> 1
- net N$24: track 17.1 -> 12.0 mm
- net N$3: track 45.9 -> 50.4 mm
- net N$11: track 61.0 -> 64.1 mm
- net N$19: track 28.8 -> 26.0 mm
- net N$26: track 16.7 -> 14.2 mm
- net N$6: track 53.0 -> 50.7 mm, vias 2 -> 0
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Other:
- board size 53.3 x 49.5 mm -> 53.3 x 49.6 mm
- board text added: "FSQCall Telemetry Rev B"
- board text added: "FSQCall Telemetry Shield Rev B"
- board text removed: "FSQCall Telemetry Shield Rev A"
