File: FSQCallTelemetry.sch (EAGLE design)
At the start: 22 parts, among them IC1 LM358, IC2 LM358, J1 1X2-3.5MM, J2 1X2-3.5MM, J3 1X2-3.5MM

Commit message: Add files via upload
Parts:
- added C3, C4: (no value), rcl:C-US050-025X075
- added JP1: (no value), jumper:JP1E
- added R13: 100K, resistor:R-US_0207/10
Connections:
- new net N$26: JP1.2, R13.1
- new net N$6: C3.1, IC1G1.V+, IC2G1.V+, U$1.VIN
- new net N$7: C4.1, U$1.AREF
- net GND: now also C3.2, C4.2, R13.2
- net N$14: now also JP1.1
- net VCC: no longer IC1G1.V+, IC2G1.V+
Other:
- note added: "0.3"
- note added: "Optional ADC Filter"
- note added: "Optional Configuration: Remove IC1 R6 = 220K Jumper across R7 Install JP1"
- note removed: "0.2"
